Commit message: Added launch files and RViz visualization

File: src/robot_description/urdf/robot.urdf (robot description, URDF)
Before this commit: robot vision_robot, 1 links, 0 joints
Links:
- added link world
Joints:
- added joint world_to_base: type fixed, parent world, child base_link, origin xyz=0 0 0

Commit message: Added LiDAR sensor to robot model

File: src/robot_description/urdf/robot.urdf (robot description, URDF)
Before this commit: robot vision_robot, 2 links, 1 joints
Links:
- added link caster_wheel; visual sphere radius=0.03
- added link left_wheel; visual cylinder length=0.02 radius=0.05
- added link lidar_link; visual cylinder length=0.05 radius=0.04
- added link right_wheel; visual cylinder length=0.02 radius=0.05
Joints:
- added joint caster_joint: type fixed, parent base_link, child caster_wheel, origin xyz=-0.15 0 0.03
- added joint left_wheel_joint: type continuous, parent base_link, child left_wheel, origin xyz=0 0.15 0.05, axis 0 1 0
- added joint lidar_joint: type fixed, parent base_link, child lidar_link, origin xyz=0 0 0.12
- added joint right_wheel_joint: type continuous, parent base_link, child right_wheel, origin xyz=0 -0.15 0.05, axis 0 1 0

Commit message: Robot motion using cmd_vel

File: src/robot_description/urdf/robot.urdf (robot description, URDF)
Before this commit: robot vision_robot, 6 links, 5 joints
Links:
- removed link world
- link left_wheel: mass None -> 0.5; geometry collision cylinder length=0.02 radius=0.05; visual cylinder length=0.02 radius=0.05
- link right_wheel: mass None -> 0.5; geometry collision cylinder length=0.02 radius=0.05; visual cylinder length=0.02 radius=0.05
Joints:
- removed joint world_to_base
